Commit message: add missing config params for moveit

File: config/srdf/teleop_arms.srdf.xacro (robot description, xacro)
@@ -1,5 +1,5 @@
 <?xml version="1.0" ?>
 <robot name="tiago_pro" xmlns:xacro="http://ros.org/wiki/xacro">
-<disable_collisions link1="arm_teleop_right_1_link" link2="arm_teleop_right_2_link" reason="Adjacent"/>
+    <disable_collisions link1="arm_teleop_right_1_link" link2="arm_teleop_right_2_link" reason="Adjacent"/>
     <disable_collisions link1="arm_teleop_right_1_link" link2="arm_teleop_right_3_link" reason="Never"/>
     <disable_collisions link1="arm_teleop_right_1_link" link2="arm_teleop_right_4_link" reason="Never"/>
@@ -117,3 +117,10 @@
     <disable_collisions link1="wrist_teleop_right_ft_sensor_base_link" link2="wrist_teleop_right_ft_tool_link" reason="Adjacent"/>
     <disable_collisions link1="wrist_teleop_right_ft_sensor_link" link2="wrist_teleop_right_ft_tool_link" reason="Never"/>
+    <disable_collisions link1="wrist_teleop_right_ft_sensor_link" link2="wrist_teleop_right_ft_tool_link" reason="Never"/>
+    <disable_collisions link1="teleop_handle_right_link" link2="arm_teleop_right_7_link" reason="Never"/>
+    <disable_collisions link1="teleop_handle_left_link" link2="arm_teleop_left_7_link" reason="Never"/>
+    <disable_collisions link1="arm_teleop_right_1_link" link2="pilot_station_base_link" reason="Adjacent"/>
+    <disable_collisions link1="arm_teleop_left_1_link" link2="pilot_station_base_link" reason="Adjacent"/>
+    <disable_collisions link1="arm_teleop_right_1_link" link2="pilot_station_arm_left_link" reason="Adjacent"/>
+    <disable_collisions link1="arm_teleop_left_1_link" link2="pilot_station_arm_right_link" reason="Adjacent"/>
 </robot>

File: config/srdf/tiago_pro.srdf.xacro (robot description, xacro)
@@ -54,4 +54,14 @@
             <group name="torso" />
         </group>
+        <group name="arm_teleop_${side}">
+            <joint name="arm_teleop_${side}_1_joint" />
+            <joint name="arm_teleop_${side}_2_joint" />
+            <joint name="arm_teleop_${side}_3_joint" />
+            <joint name="arm_teleop_${side}_4_joint" />
+            <joint name="arm_teleop_${side}_5_joint" />
+            <joint name="arm_teleop_${side}_6_joint" />
+            <joint name="arm_teleop_${side}_7_joint" />
+            <!-- <joint name="arm_teleop_${side}_tool_joint" /> -->
+        </group>
     </xacro:macro>
     <xacro:if value="${has_arm_left}">
@@ -66,4 +76,11 @@
             <group name="arm_right" />
             <group name="arm_left" />
+        </group>
+    </xacro:if>
+    <!-- if has_teleop create a group arm with arm_teleop_left and arm_teleop right -->
+    <xacro:if value="${has_teleop_arms}">
+        <group name="arms_teleop">
+            <group name="arm_teleop_left" />
+            <group name="arm_teleop_right" />
         </group>
     </xacro:if>
